Commit message: 批量生成

File: robot_assets/generated_robot.urdf (robot description, URDF)
Before this commit: robot generated_multileg, 61 links, 60 joints
Links:
- removed link leg_8_foot
- removed link leg_8_hip
- removed link leg_8_knee
- removed link leg_8_lower
- removed link leg_8_swing_node
- removed link leg_8_upper
- removed link leg_9_foot
- removed link leg_9_hip
- removed link leg_9_knee
- removed link leg_9_lower
- removed link leg_9_swing_node
- removed link leg_9_upper
- link base_link: mass 43.018476929 -> 34.659569688
Joints:
- removed joint leg_8_drop
- removed joint leg_8_foot_mount
- removed joint leg_8_knee_mount
- removed joint leg_8_lift
- removed joint leg_8_mount
- removed joint leg_8_swing
- removed joint leg_9_drop
- removed joint leg_9_foot_mount
- removed joint leg_9_knee_mount
- removed joint leg_9_lift
- removed joint leg_9_mount
- removed joint leg_9_swing
- joint leg_0_drop: axis 1.000000000 0.000000000 0.000000000 -> 0.789875134 0.613267700 0.000000000
- joint leg_0_foot_mount: origin xyz=0.000577223 0.025544406 -0.298909936 rpy=0.000000000 0.000000000 0.000000000 -> xyz=0.041672985 -0.023595685 -0.296153011 rpy=0.000000000 0.000000000 0.000000000
- joint leg_0_knee_mount: origin xyz=0.065253293 0.054708047 -0.266737769 rpy=0.000000000 0.000000000 0.000000000 -> xyz=0.005686805 -0.278118381 -0.031903393 rpy=0.000000000 0.000000000 0.000000000
- joint leg_0_lift: axis 1.000000000 0.000000000 0.000000000 -> 0.789875134 0.613267700 0.000000000
- joint leg_0_mount: origin xyz=-0.131024023 -0.220000000 -0.090000000 rpy=0.000000000 0.000000000 0.000000000 -> xyz=0.115208324 -0.252166135 -0.090000000 rpy=0.000000000 0.000000000 0.000000000
- joint leg_1_drop: axis 1.000000000 0.000000000 0.000000000 -> -0.411068534 0.911604443 0.000000000
- joint leg_1_foot_mount: origin xyz=-0.008351710 0.022418430 -0.299044584 rpy=0.000000000 0.000000000 0.000000000 -> xyz=0.047236951 0.001979701 -0.296251162 rpy=0.000000000 0.000000000 0.000000000
- joint leg_1_knee_mount: origin xyz=-0.021002291 0.056376286 -0.273460451 rpy=0.000000000 0.000000000 0.000000000 -> xyz=0.131331517 0.245240502 -0.031766786 rpy=0.000000000 0.000000000 0.000000000
- joint leg_1_lift: axis 1.000000000 0.000000000 0.000000000 -> -0.411068534 0.911604443 0.000000000
- joint leg_1_mount: origin xyz=0.085489387 -0.220000000 -0.090000000 rpy=0.000000000 0.000000000 0.000000000 -> xyz=0.259942467 0.216558427 -0.090000000 rpy=0.000000000 0.000000000 0.000000000
- joint leg_1_swing: limit lower=-0.120000000 upper=0.120000000 effort=20.000000000 velocity=2.000000000 -> lower=-0.550000000 upper=0.550000000 effort=20.000000000 velocity=2.000000000
- joint leg_2_drop: axis 0.971934458 0.235251799 0.000000000 -> -0.411068534 0.911604443 0.000000000
- joint leg_2_foot_mount: origin xyz=-0.009950645 0.020697439 -0.299119710 rpy=0.000000000 0.000000000 0.000000000 -> xyz=0.012518463 0.069978466 -0.291455490 rpy=0.000000000 0.000000000 0.000000000
- joint leg_2_knee_mount: origin xyz=-0.083209987 0.029128831 -0.265758555 rpy=0.000000000 0.000000000 0.000000000 -> xyz=0.224788506 0.161576310 -0.041990757 rpy=0.000000000 0.000000000 0.000000000
- joint leg_2_lift: axis 0.971934458 0.235251799 0.000000000 -> -0.411068534 0.911604443 0.000000000
- joint leg_2_mount: origin xyz=0.300537158 -0.207714671 -0.090000000 rpy=0.000000000 0.000000000 0.000000000 -> xyz=0.238331579 0.264483722 -0.090000000 rpy=0.000000000 0.000000000 0.000000000
- joint leg_3_drop: axis 0.000000000 1.000000000 0.000000000 -> -0.959884293 -0.280396404 0.000000000
- joint leg_3_foot_mount: origin xyz=-0.023782836 0.002591088 -0.299044584 rpy=0.000000000 0.000000000 0.000000000 -> xyz=-0.013004581 0.032615023 -0.297938150 rpy=0.000000000 0.000000000 0.000000000
- joint leg_3_knee_mount: origin xyz=-0.059807400 0.006515886 -0.273460451 rpy=0.000000000 0.000000000 0.000000000 -> xyz=0.170750294 0.219916874 -0.029680052 rpy=0.000000000 0.000000000 0.000000000
- joint leg_3_lift: axis 0.000000000 1.000000000 0.000000000 -> -0.959884293 -0.280396404 0.000000000
- joint leg_3_mount: origin xyz=0.360000000 -0.037988471 -0.090000000 rpy=0.000000000 0.000000000 0.000000000 -> xyz=0.183386223 0.268544448 -0.090000000 rpy=0.000000000 0.000000000 0.000000000
- joint leg_3_swing: limit lower=-0.120000000 upper=0.120000000 effort=20.000000000 velocity=2.000000000 -> lower=-0.550000000 upper=0.550000000 effort=20.000000000 velocity=2.000000000
- joint leg_4_drop: axis -0.668216856 0.743966554 0.000000000 -> 0.335939219 -0.941883667 0.000000000
- joint leg_4_foot_mount: origin xyz=-0.036534817 -0.002331257 -0.297757909 rpy=0.000000000 0.000000000 0.000000000 -> xyz=-0.058323705 0.036854707 -0.291959031 rpy=0.000000000 0.000000000 0.000000000
- joint leg_4_knee_mount: origin xyz=-0.036524783 -0.053747182 -0.272354880 rpy=0.000000000 0.000000000 0.000000000 -> xyz=-0.268049090 -0.070123954 -0.040401939 rpy=0.000000000 0.000000000 0.000000000
- joint leg_4_lift: axis -0.668216856 0.743966554 0.000000000 -> 0.335939219 -0.941883667 0.000000000
- joint leg_4_mount: origin xyz=0.341098952 0.171282828 -0.090000000 rpy=0.000000000 0.000000000 0.000000000 -> xyz=-0.239859929 0.011547865 -0.090000000 rpy=0.000000000 0.000000000 0.000000000
- joint leg_5_drop: axis -1.000000000 0.000000000 0.000000000 -> 0.335939219 -0.941883667 0.000000000
- joint leg_5_foot_mount: origin xyz=-0.013082017 -0.020029924 -0.299044584 rpy=0.000000000 0.000000000 0.000000000 -> xyz=-0.058396156 0.036105606 -0.292038138 rpy=0.000000000 0.000000000 0.000000000
- joint leg_5_knee_mount: origin xyz=-0.032897735 -0.050369842 -0.273460451 rpy=0.000000000 0.000000000 0.000000000 -> xyz=-0.266869256 -0.074613987 -0.040169056 rpy=0.000000000 0.000000000 0.000000000
- joint leg_5_lift: axis -1.000000000 0.000000000 0.000000000 -> 0.335939219 -0.941883667 0.000000000
- joint leg_5_mount: origin xyz=0.146311702 0.220000000 -0.090000000 rpy=0.000000000 0.000000000 0.000000000 -> xyz=-0.238165856 0.006798139 -0.090000000 rpy=0.000000000 0.000000000 0.000000000
- joint leg_5_swing: limit lower=-0.120000000 upper=0.120000000 effort=20.000000000 velocity=2.000000000 -> lower=-0.550000000 upper=0.550000000 effort=20.000000000 velocity=2.000000000
- joint leg_6_drop: axis -1.000000000 0.000000000 0.000000000 -> 0.335939219 -0.941883667 0.000000000
- joint leg_6_foot_mount: origin xyz=0.024339412 -0.028225878 -0.297675818 rpy=0.000000000 0.000000000 0.000000000 -> xyz=-0.057741550 0.023326344 -0.293465151 rpy=0.000000000 0.000000000 0.000000000
- joint leg_6_knee_mount: origin xyz=-0.011937681 -0.062074605 -0.272771397 rpy=0.000000000 0.000000000 0.000000000 -> xyz=-0.237541679 -0.143651501 -0.036581373 rpy=0.000000000 0.000000000 0.000000000
- joint leg_6_lift: axis -1.000000000 0.000000000 0.000000000 -> 0.335939219 -0.941883667 0.000000000
- joint leg_6_mount: origin xyz=-0.070201708 0.220000000 -0.090000000 rpy=0.000000000 0.000000000 0.000000000 -> xyz=-0.211984730 -0.066606732 -0.090000000 rpy=0.000000000 0.000000000 0.000000000
- joint leg_7_drop: axis -1.000000000 0.000000000 0.000000000 -> 0.335939219 -0.941883667 0.000000000
- joint leg_7_foot_mount: origin xyz=0.038540715 -0.017906143 -0.296974718 rpy=0.000000000 0.000000000 0.000000000 -> xyz=-0.029777178 -0.054914311 -0.293424161 rpy=0.000000000 0.000000000 0.000000000
- joint leg_7_knee_mount: origin xyz=0.019755023 -0.040000737 -0.276423009 rpy=0.000000000 0.000000000 0.000000000 -> xyz=-0.274533916 -0.041065644 -0.036670725 rpy=0.000000000 0.000000000 0.000000000
- joint leg_7_lift: axis -1.000000000 0.000000000 0.000000000 -> 0.335939219 -0.941883667 0.000000000
- joint leg_7_mount: origin xyz=-0.286715118 0.220000000 -0.090000000 rpy=0.000000000 0.000000000 0.000000000 -> xyz=-0.188328386 -0.132932790 -0.090000000 rpy=0.000000000 0.000000000 0.000000000
